File: pcb/reflow-oven-controller/reflow-oven-controller.kicad_pcb (KiCad board)
At the start: 2 copper layers, 68 parts, among them J1 12V_IN, J10 RELAY_4, J11 RELAY_5, J12 RELAY_6, J13 RELAY_7, J14 DISPLAY, J2 USB, J3 TEMP_0, J4 TEMP_1, J5 DEBUG, J6 GPIO, J7 RELAY_1, J8 RELAY_2, J9 RELAY_3, Q1 AO3400A, U1 TPS5430DDA, U2 AMS1117-3.3, U3 RP2040, U4 MAX31855KASA, U5 MAX31855KASA, U6 W25Q128JVS, U7 ULN2003A, Y1 X322512MSB4SI

Commit message: Finish PCB
Parts:
- removed J13: RELAY_7, TerminalBlock_MetzConnect:TerminalBlock_MetzConnect_Type059_RT06302HBWC_1x02_P3.50mm_Horizontal
- removed J5: DEBUG, Connector_PinHeader_2.54mm:PinHeader_1x03_P2.54mm_Vertical
- removed J6: GPIO, Connector_PinHeader_2.54mm:PinHeader_2x07_P2.54mm_Vertical
- removed JP1: BOOT, Connector_PinHeader_2.54mm:PinHeader_1x02_P2.54mm_Vertical
- removed JP2: RESET, Connector_PinHeader_2.54mm:PinHeader_1x02_P2.54mm_Vertical
- removed Q1: AO3400A, Package_TO_SOT_SMD:SOT-23
- removed the R13 at (146.9, 81.5)
- added D4: LED, LED_SMD:LED_0603_1608Metric, F.Cu at (85.7, 84.5)
- added H1: MountingHole, MountingHole:MountingHole_3.2mm_M3, F.Cu at (74.0, 146.0)
- added H2: MountingHole, MountingHole:MountingHole_3.2mm_M3, F.Cu at (121.0, 146.0)
- added H3: MountingHole, MountingHole:MountingHole_3.2mm_M3, F.Cu at (74.0, 54.0)
- added H4: MountingHole, MountingHole:MountingHole_3.2mm_M3, F.Cu at (121.0, 54.0)
- added R15: 0R, Resistor_SMD:R_0603_1608Metric, F.Cu at (87.4, 126.5)
- D2, D3: value M7 -> SS34
- J11: value RELAY_5 -> RELAY_OPT; footprint TerminalBlock_MetzConnect:TerminalBlock_MetzConnect_Type059_RT06302HBWC_1x02_P3.50mm_Horizontal -> Connector_PinHeader_2.54mm:PinHeader_2x04_P2.54mm_Vertical_SMD
- J12: value RELAY_6 -> HEADER; footprint TerminalBlock_MetzConnect:TerminalBlock_MetzConnect_Type059_RT06302HBWC_1x02_P3.50mm_Horizontal -> Connector_PinHeader_2.54mm:PinHeader_2x10_P2.54mm_Vertical_SMD
- J2: footprint Connector_USB:USB_C_Receptacle_GCT_USB4115-03-C -> lib:GCT_USB4145-03-0070-C_REVA2; moved to B.Cu
- J3: value TEMP_0 -> TEMP_1
- J4: value TEMP_1 -> TEMP_2
- R14: value 10k -> 470R
- moved J2 117.2 mm to (83.2, 146.1), turned to 0 degrees
- moved R7 95.3 mm to (90.6, 91.2)
- moved R8 94.8 mm to (90.6, 89.6)
- moved J14 90.9 mm to (97.5, 122.5)
- moved L1 87.9 mm to (76.8, 73.5)
- moved C3 86.1 mm to (84.6, 73.5)
- moved R2 85.0 mm to (79.8, 143.1), turned to 180 degrees
- moved R1 83.8 mm to (86.6, 143.1), turned to 0 degrees
- moved D2 78.4 mm to (74.0, 83.3)
- moved D3 75.0 mm to (74.0, 90.6), turned to -90 degrees
- moved D1 74.4 mm to (75.6, 65.3), turned to -90 degrees
- moved R3 71.2 mm to (84.1, 69.3)
- moved U5 71.2 mm to (112.3, 132.7)
- moved C16 69.2 mm to (86.8, 95.6), turned to -90 degrees
- moved J7 68.4 mm to (92.2, 56.0), turned to 180 degrees
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Connections:
- net /USB_DM renamed /USB_D-
- net /USB_DP renamed /USB_D+
- D3 pad 2: Net-(D3-Pad2) -> Net-(J2-PadA4)
- J1 pad 1: +12V -> GND
- J1 pad 2: GND -> +12V
- J11 pad 1: +12V -> Net-(J11-Pad1)
- J11 pad 2: Net-(J11-Pad2) -> +12V
- J12 pad 1: +12V -> +3.3V
- J12 pad 2: Net-(J12-Pad2) -> /GPIO11
- J14 pad 39: +3.3V -> Net-(J14-Pad39)
- J2 pad A4: Net-(D3-Pad2) -> Net-(J2-PadA4)
- J2 pad A9: Net-(D3-Pad2) -> Net-(J2-PadA4)
- J2 pad B4: Net-(D3-Pad2) -> Net-(J2-PadA4)
- J2 pad B9: Net-(D3-Pad2) -> Net-(J2-PadA4)
- J3 pad 1: Net-(C6-Pad1) -> Net-(C6-Pad2)
- J3 pad 2: Net-(C6-Pad2) -> Net-(C6-Pad1)
- J4 pad 1: Net-(C7-Pad1) -> Net-(C7-Pad2)
- J4 pad 2: Net-(C7-Pad2) -> Net-(C7-Pad1)
- R13 pad 2: Net-(U3-Pad26) -> /RESET
- R14 pad 1: Net-(D3-Pad2) -> +3.3V
- R9 pad 1: Net-(JP1-Pad2) -> /BOOT
- U3 pad 11: /RELAY1 -> /SPI_CS0
- U3 pad 12: /RELAY2 -> /LCD_RESET
- U3 pad 13: /RELAY3 -> /GPIO1
- U3 pad 14: /RELAY4 -> /GPIO2
- U3 pad 15: /RELAY5 -> /GPIO3
- U3 pad 16: /RELAY6 -> /GPIO4
- U3 pad 17: /RELAY7 -> /GPIO5
- U3 pad 18: /GPIO1 -> /GPIO6
- U3 pad 2: /SPI_SCK -> /TOUCH_XL
- U3 pad 24: Net-(J5-Pad1) -> /SWCLK
- U3 pad 25: Net-(J5-Pad2) -> /SWD
- U3 pad 26: Net-(U3-Pad26) -> /RESET
- U3 pad 27: /GPIO2 -> /GPIO7
- U3 pad 28: /GPIO3 -> /GPIO8
- U3 pad 29: /GPIO4 -> /GPIO9
- U3 pad 3: /SPI_MISO -> /TOUCH_YD
- U3 pad 30: /GPIO5 -> /RELAY7
- U3 pad 31: /GPIO6 -> /RELAY6
- U3 pad 32: /GPIO7 -> /RELAY5
- U3 pad 34: /GPIO8 -> /RELAY4
- U3 pad 35: /GPIO9 -> /RELAY3
- U3 pad 36: /TOUCH_XL -> /RELAY2
- U3 pad 37: /TOUCH_YD -> /RELAY1
- U3 pad 38: /TOUCH_YU -> /GPIO10
- U3 pad 39: /TOUCH_XR -> /GPIO11
- U3 pad 4: /SPI_MOSI -> /SPI_CS2
- U3 pad 40: /GPIO10 -> /TOUCH_YU
- U3 pad 41: /GPIO11 -> /TOUCH_XR
- U3 pad 5: /SPI_CS0 -> /LCD_A0
- U3 pad 6: /SPI_CS1 -> /SPI_MOSI
- U3 pad 7: /SPI_CS2 -> /SPI_MISO
- U3 pad 8: /LCD_A0 -> /SPI_SCK
- U3 pad 9: /LCD_RESET -> /SPI_CS1
- U7 pad 10: Net-(J13-Pad2) -> Net-(J11-Pad5)
- U7 pad 11: Net-(J12-Pad2) -> Net-(J11-Pad3)
- U7 pad 12: Net-(J11-Pad2) -> Net-(J11-Pad1)
Routing:
- net /USB_D-: track 0.00 -> 68.8 mm, vias 0 -> 3
- net /LCD_RESET: track 0.00 -> 68.7 mm
- net /USB_D+: track 0.00 -> 67.9 mm, vias 0 -> 1
- net /SPI_SCK: track 0.00 -> 66.5 mm, vias 0 -> 2
- net GND: track 0.00 -> 63.9 mm, vias 0 -> 35
- net /SPI_MISO: track 0.00 -> 60.7 mm
- net /SPI_CS0: track 0.00 -> 58.6 mm
- net /TOUCH_YU: track 0.00 -> 55.1 mm, vias 0 -> 2
- net /TOUCH_XR: track 0.00 -> 53.7 mm, vias 0 -> 2
- net /SPI_MOSI: track 0.00 -> 52.9 mm
- net /LCD_A0: track 0.00 -> 50.6 mm
- net /SPI_CS2: track 0.00 -> 49.0 mm
- net /SPI_CS1: track 0.00 -> 48.6 mm
- net /TOUCH_YD: track 0.00 -> 45.8 mm
- net /TOUCH_XL: track 0.00 -> 42.3 mm
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- added copper zone on F.Cu, net +12V
- added copper zone on F.Cu, net +3.3V
- added copper zone on B.Cu, net GND
- added copper zone on F.Cu, net GND
- added copper zone on F.Cu, net Net-(C2-Pad2)
- added copper zone on F.Cu, net Net-(C3-Pad1)
- added copper zone on F.Cu, net Net-(C4-Pad1)
- added copper zone on F.Cu, net Net-(J2-PadA4)
Other:
- board outline added: 55 x 100 mm
- board text added: "+ 12V -"
- board text added: "- T1 +"
- board text added: "- T2 +"
- board text added: "12V"
- board text added: "3V3"
- board text added: "BOOT"
- board text added: "GND"
- board text added: "IO1"
- board text added: "IO10"
- board text added: "IO11"
- board text added: "IO2"
- board text added: "IO3"
- board text added: "IO4"
- board text added: "IO5"
- board text added: "IO6"
- board text added: "IO7"
- board text added: "IO8"
- board text added: "IO9"
- board text added: "REL1 +"
- board text added: "REL2 +"
- board text added: "REL3 +"
- board text added: "REL4 +"
- board text added: "REL5"
- board text added: "REL6"
- board text added: "REL7"
- board text added: "RST"
- board text added: "SWCL"
- board text added: "SWD"
