File: pcb/reflow-oven-controller/reflow-oven-controller.kicad_sch (KiCad schematic)
At the start: 67 parts, among them J1 12V_IN, J10 RELAY_4, J11 RELAY_5, J12 RELAY_6, J13 RELAY_7, J14 DISPLAY, J2 USB, J3 TEMP_0, J4 TEMP_1, J5 DEBUG, J6 GPIO, J7 RELAY_1, J8 RELAY_2, J9 RELAY_3, U1 TPS5430DDA, U2 AMS1117-3.3, U3 RP2040, U4 MAX31855KASA, U5 MAX31855KASA, U6 W25Q128JVS, U7 ULN2003A, Y1 X322512MSB4SI

Commit message: Finish PCB
Parts:
- removed D2, D3: M7, Diode_SMD:D_SMA, symbol Device:D
- removed J11: RELAY_5, TerminalBlock_MetzConnect:TerminalBlock_MetzConnect_Type059_RT06302HBWC_1x02_P3.50mm_Horizontal, symbol Connector_Generic:Conn_01x02
- removed J12: RELAY_6, TerminalBlock_MetzConnect:TerminalBlock_MetzConnect_Type059_RT06302HBWC_1x02_P3.50mm_Horizontal, symbol Connector_Generic:Conn_01x02
- removed J13: RELAY_7, TerminalBlock_MetzConnect:TerminalBlock_MetzConnect_Type059_RT06302HBWC_1x02_P3.50mm_Horizontal, symbol Connector_Generic:Conn_01x02
- removed J5: DEBUG, Connector_PinHeader_2.54mm:PinHeader_1x03_P2.54mm_Vertical, symbol Connector_Generic:Conn_01x03
- removed J6: GPIO, Connector_PinHeader_2.54mm:PinHeader_2x07_P2.54mm_Vertical, symbol Connector_Generic:Conn_02x07_Odd_Even
- removed JP1: BOOT, Connector_PinHeader_2.54mm:PinHeader_1x02_P2.54mm_Vertical, symbol Jumper:Jumper_2_Open
- removed JP2: RESET, Connector_PinHeader_2.54mm:PinHeader_1x02_P2.54mm_Vertical, symbol Jumper:Jumper_2_Open
- added D2, D3: SS34, Diode_SMD:D_SMA, symbol Device:D_Schottky
- added H1, H2, H3, H4: MountingHole, MountingHole:MountingHole_3.2mm_M3, symbol Mechanical:MountingHole
- added J11: RELAY_OPT, Connector_PinHeader_2.54mm:PinHeader_2x04_P2.54mm_Vertical_SMD, symbol Connector_Generic:Conn_02x04_Odd_Even
- added J12: HEADER, Connector_PinHeader_2.54mm:PinHeader_2x10_P2.54mm_Vertical_SMD, symbol Connector_Generic:Conn_02x10_Odd_Even
- added R15: 0R, Resistor_SMD:R_0603_1608Metric, symbol Device:R
- J1, J10, J7, J8, J9: symbol Connector_Generic:Conn_01x02 -> Connector:Screw_Terminal_01x02
- J2: footprint USB_C_Receptacle_GCT_USB4115-03-C -> lib:GCT_USB4145-03-0070-C_REVA2; LCSC C381139 -> -
- J3: value TEMP_0 -> TEMP_1; symbol Connector_Generic:Conn_01x02 -> Connector:Screw_Terminal_01x02
- J4: value TEMP_1 -> TEMP_2; symbol Connector_Generic:Conn_01x02 -> Connector:Screw_Terminal_01x02
- L1: Current 1.2A -> (none)
Connections:
- net +12V: now also J1.2 (Pin_2), J11.2 (Pin_2), J11.4 (Pin_4), J11.6 (Pin_6), J11.8 (Pin_8); no longer J1.1 (Pin_1)
- net +3.3V: now also J12.1 (Pin_1), R15.1; no longer J14.39 (Pin_39)
- net GND: now also J1.1 (Pin_1), J11.7 (Pin_7), J12.10 (Pin_10), J12.12 (Pin_12), J12.20 (Pin_20), J12.8 (Pin_8); no longer J1.2 (Pin_2)
- net GPIO1: now also U3.13 (GPIO10), J12.18 (Pin_18); no longer U3.18 (GPIO15)
- net GPIO10: now also U3.38 (GPIO26_ADC0), J12.3 (Pin_3); no longer U3.40 (GPIO28_ADC2)
- net GPIO11: now also U3.39 (GPIO27_ADC1), J12.2 (Pin_2); no longer U3.41 (GPIO29_ADC3)
- net GPIO2: now also U3.14 (GPIO11), J12.17 (Pin_17); no longer U3.27 (GPIO16)
- net GPIO3: now also U3.15 (GPIO12), J12.16 (Pin_16); no longer U3.28 (GPIO17)
- net GPIO4: now also U3.16 (GPIO13), J12.15 (Pin_15); no longer U3.29 (GPIO18)
- net GPIO5: now also U3.17 (GPIO14), J12.14 (Pin_14); no longer U3.30 (GPIO19)
- net GPIO6: now also U3.18 (GPIO15), J12.13 (Pin_13); no longer U3.31 (GPIO20)
- net GPIO7: now also U3.27 (GPIO16), J12.6 (Pin_6); no longer U3.32 (GPIO21)
- net GPIO8: now also U3.28 (GPIO17), J12.5 (Pin_5); no longer U3.34 (GPIO22)
- net GPIO9: now also U3.29 (GPIO18), J12.4 (Pin_4); no longer U3.35 (GPIO23)
- net LCD_A0: now also U3.5 (GPIO3); no longer U3.8 (GPIO6)
- net LCD_RESET: now also U3.12 (GPIO9); no longer U3.9 (GPIO7)
- net RELAY1: now also U3.37 (GPIO25); no longer U3.11 (GPIO8)
- net RELAY2: now also U3.36 (GPIO24); no longer U3.12 (GPIO9)
- net RELAY3: now also U3.35 (GPIO23); no longer U3.13 (GPIO10)
- net RELAY4: now also U3.34 (GPIO22); no longer U3.14 (GPIO11)
- net RELAY5: now also U3.32 (GPIO21); no longer U3.15 (GPIO12)
- net RELAY6: now also U3.31 (GPIO20); no longer U3.16 (GPIO13)
- net RELAY7: now also U3.30 (GPIO19); no longer U3.17 (GPIO14)
- net SPI_CS0: now also U3.11 (GPIO8); no longer U3.5 (GPIO3)
- net SPI_CS1: now also U3.9 (GPIO7); no longer U3.6 (GPIO4)
- net SPI_CS2: now also U3.4 (GPIO2); no longer U3.7 (GPIO5)
- net SPI_MISO: now also U3.7 (GPIO5); no longer U3.3 (GPIO1)
- net SPI_MOSI: now also U3.6 (GPIO4); no longer U3.4 (GPIO2)
- net SPI_SCK: now also U3.8 (GPIO6); no longer U3.2 (GPIO0)
- net TOUCH_XL: now also U3.2 (GPIO0); no longer U3.36 (GPIO24)
- net TOUCH_XR: now also U3.41 (GPIO29_ADC3); no longer U3.39 (GPIO27_ADC1)
- net TOUCH_YD: now also U3.3 (GPIO1); no longer U3.37 (GPIO25)
- net TOUCH_YU: now also U3.40 (GPIO28_ADC2); no longer U3.38 (GPIO26_ADC0)
- net at C7.1, U5.3 (T+): now also J4.2 (Pin_2); no longer J4.1 (Pin_1)
- net at C7.2, R6.1, U5.2 (T-): now also J4.1 (Pin_1); no longer J4.2 (Pin_2)
- net at C6.1, U4.3 (T+): now also J3.2 (Pin_2); no longer J3.1 (Pin_1)
- net at C6.2, R5.1, U4.2 (T-): now also J3.1 (Pin_1); no longer J3.2 (Pin_2)
- net at U7.10 (O7): now also J11.5 (Pin_5)
- net RESET: now reaches R13.2, U3.26 (RUN)
- net RESET: now also J12.7 (Pin_7)
- net at C3.1, L1.2, R3.1: now also D2.2 (A)
- net at U7.11 (O6): now also J11.3 (Pin_3)
- net SWCLK: now reaches U3.24 (SWCLK)
- net SWCLK: now also J12.11 (Pin_11)
- net SWD: now reaches U3.25 (SWD)
- net SWD: now also J12.9 (Pin_9)
- net at C4.1, U2.3 (VI): now also D2.1 (K), D3.1 (K)
- net BOOT: now reaches R9.1
- net BOOT: now also J12.19 (Pin_19)
- net at U7.12 (O5): now also J11.1 (Pin_1)
- net at J2.A4 (VBUS), J2.A9 (VBUS), J2.B4 (VBUS)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: now also D3.2 (A)
- net USB_DM renamed USB_D-
- net USB_DP renamed USB_D+
- new net: J14.39 (Pin_39), R15.2
Other:
- moved on the sheet: C15, C16, R11, R13, R9, U6
